File: 1.INV_KiCAD/VCUinvertor.kicad_sch (KiCad schematic)
At the start: 117 parts, among them J7 PowerSupply, J9 BRAKE LIGHT, K1 IM06, Q1 2N7002, Q10 2N7002, Q13 BC848C, Q2 2N7002, Q3 2N7002, Q4 2N7002, Q5 2N7002, Q6 2N7002, Q7 2N7002, Q8 2N7002, Q9 2N7002, U1 TJA1448ATK, U2 REF3433T, U3 TLV76150DCY

Commit message: Block diagram cleanUp
Parts:
- K1: value IM06 -> IM06DGR
Other:
- moved on the sheet: D2, J7, J9, JO16, JO17, JO18, JO2, JO20, JO36, Q13, R31, VCC_BAT1

Commit message: Relay NC to NO change
Connections:
- net BAT+: now also K1.4; no longer K1.2
- net NXP_TPSOUT01: now also NXP11.1 (Pin_1); no longer NXP14.1 (Pin_1)
- net NXP_TPSOUT02: now also NXP11.4 (Pin_4); no longer NXP14.3 (Pin_3)
Other:
- note added: "1. Switch The switch to NO from NC --> From pin 2 to pin 4 2.Move the connectors of the TPS OUT1 & 2"
- moved on the sheet: R32
