File: 1.INV_KiCAD/VCUinvertor.kicad_pcb (KiCad board)
At the start: 2 copper layers, 100.7 x 117.9 mm, 118 parts, among them J7 PowerSupply, J9 BRAKE LIGHT, K1 IM06DGR, Q1 2N7002, Q10 2N7002, Q13 BC848C, Q2 2N7002, Q3 2N7002, Q4 2N7002, Q5 2N7002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

Commit message: Error corrections - Done
Parts:
- moved C10 0.36 mm to (119.5, 84.1)
- moved R28 0.30 mm to (120.8, 121.6)
- moved C9 0.26 mm to (117.2, 84.1)
Routing:
- net unconnected-(K1-Pad2): track 1.15 -> 0.00 mm
- net GND: track 86.0 -> 86.5 mm
Changed lines of the file:
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@@
 	(footprint "Capacitor_SMD:C_1206_3216Metric_Pad1.33x1.80mm_HandSolder"
 		(layer "F.Cu")
-		(at 117.46301 84.09274 90)
+		(at 117.20051 84.09274 90)
 		(descr "Capacitor SMD 1206 (3216 Metric), square (rectangular) end terminal, IPC-7351 nominal with elongated pad for handsoldering. (Body size source: IPC-SM-782 page 76, https://www.pcb-3d.com/wordpress/wp-content/uploads/ipc-sm-782a_amendment_1_and_2.pdf), generated with kicad-footprint-generator")
 		(tags "capacitor handsolder")
@@
 	(footprint "Capacitor_SMD:C_1206_3216Metric_Pad1.33x1.80mm_HandSolder"
 		(layer "F.Cu")
-		(at 119.86301 84.09274 90)
+		(at 119.50051 84.09274 90)
 		(descr "Capacitor SMD 1206 (3216 Metric), square (rectangular) end terminal, IPC-7351 nominal with elongated pad for handsoldering. (Body size source: IPC-SM-782 page 76, https://www.pcb-3d.com/wordpress/wp-content/uploads/ipc-sm-782a_amendment_1_and_2.pdf), generated with kicad-footprint-generator")
 		(tags "capacitor handsolder")
@@
 	(footprint "Resistor_SMD:R_1206_3216Metric_Pad1.30x1.75mm_HandSolder"
 		(layer "F.Cu")
-		(at 120.70051 121.29274)
+		(at 120.75051 121.59274)
 		(descr "Resistor SMD 1206 (3216 Metric), square (rectangular) end terminal, IPC-7351 nominal with elongated pad for handsoldering. (Body size source: IPC-SM-782 page 72, https://www.pcb-3d.com/wordpress/wp-content/uploads/ipc-sm-782a_amendment_1_and_2.pdf)")
 		(tags "resistor handsolder")
@@
 		(tags "SOT TO_SOT_SMD")
 		(property "Reference" "Q10"
-			(at 0.025 2.51 0)
+			(at 1.522645 2.217626 90)
 			(layer "F.SilkS")
 			(effects
@@
 		(fp_poly
 			(pts
-				(xy -5.400001 -1.32) (xy 4.6 -1.32) (xy 4.6 5.68) (xy -5.4 5.68)
+				(xy -4.5 1.28) (xy -3.8 1.28) (xy -3.8 3.18) (xy -4.5 3.18)
 			)
 			(stroke
 				(width 0.1)
-				(type default)
+				(type solid)
 			)
-			(fill no)
+			(fill yes)
 			(layer "F.SilkS")
 		)
 		(fp_poly
 			(pts
-				(xy -4.5 1.28) (xy -3.8 1.28) (xy -3.8 3.18) (xy -4.5 3.18)
+				(xy -5.400001 -1.32) (xy 4.6 -1.32) (xy 4.6 5.68) (xy -5.4 5.68)
 			)
 			(stroke
@@
 				(type solid)
 			)
-			(fill yes)
-			(layer "F.SilkS")
+			(fill no)
+			(layer "F.Paste")
 		)
 		(fp_text user "${REFERENCE}"
@@
 	)
 	(segment
+		(start 120.80051 115.49274)
+		(end 122.10051 114.19274)
+		(width 0.2)
+		(layer "F.Cu")
+		(net "GND")
+	)
+	(segment
 		(start 128.742865 137.010114)
 		(end 128.827355 137.010114)
@@
 	)
 	(segment
+		(start 122.30051 121.59274)
+		(end 122.30051 121.44274)
+		(width 0.2)
+		(layer "F.Cu")
+		(net "GND")
+	)
+	(segment
+		(start 119.50051 81.49274)
+		(end 119.50051 82.23024)
+		(width 0.2)
+		(layer "F.Cu")
+		(net "GND")
+	)
+	(segment
 		(start 103.68426 74.18899)
 		(end 102.98227 73.487)
@@
 	)
 	(segment
-		(start 120.80051 115.49274)
-		(end 122.10051 114.19274)
+		(start 122.10051 114.19274)
+		(end 122.10051 113.99274)
 		(width 0.2)
 		(layer "F.Cu")
@@
 	)
 	(segment
-		(start 122.10051 114.19274)
-		(end 122.10051 113.99274)
+		(start 119.50051 82.23024)
+		(end 119.80051 82.53024)
 		(width 0.2)
 		(layer "F.Cu")
@@
 	)
 	(segment
-		(start 119.86301 82.53024)
-		(end 119.41301 82.53024)
+		(start 122.30051 121.44274)
+		(end 120.80051 119.94274)
 		(width 0.2)
 		(layer "F.Cu")
@@
 	)
 	(segment
-		(start 117.46301 82.53024)
-		(end 119.86301 82.53024)
+		(start 119.85051 81.14274)
+		(end 119.50051 81.49274)
 		(width 0.2)
 		(layer "F.Cu")
@@
 	)
 	(segment
-		(start 131.10051 86.79274)
-		(end 132.53801 86.79274)
-		(width 0.2)
-		(layer "F.Cu")
-		(net "GND")
-	)
-	(segment
 		(start 126.59785 106.17394)
 		(end 126.59785 105.59008)
@@
 	)
 	(segment
-		(start 120.80051 119.69274)
-		(end 120.80051 115.49274)
+		(start 119.80051 82.53024)
+		(end 119.50051 82.53024)
+		(width 0.2)
+		(layer "F.Cu")
+		(net "GND")
+	)
+	(segment
+		(start 119.50051 82.53024)
+		(end 119.41301 82.53024)
 		(width 0.2)
 		(layer "F.Cu")
@@
 	)
 	(segment
+		(start 131.10051 86.79274)
+		(end 132.00051 86.79274)
+		(width 0.2)
+		(layer "F.Cu")
+		(net "GND")
+	)
+	(segment
 		(start 128.72551 144.49274)
 		(end 128.875 144.49274)
@@
 	)
 	(segment
-		(start 119.86301 81.15524)
-		(end 119.86301 82.53024)
+		(start 132.00051 86.79274)
+		(end 132.45051 86.34274)
 		(width 0.2)
 		(layer "F.Cu")
@@
 	)
 	(segment
+		(start 117.20051 82.53024)
+		(end 119.50051 82.53024)
+		(width 0.2)
+		(layer "F.Cu")
+		(net "GND")
+	)
+	(segment
 		(start 124.100511 55.092741)
 		(end 128.90051 59.89274)
@@
 	)
 	(segment
-		(start 119.85051 81.14274)
-		(end 119.86301 81.15524)
-		(width 0.2)
-		(layer "F.Cu")
-		(net "GND")
-	)
-	(segment
 		(start 129.15051 62.59274)
 		(end 129.30051 62.44274)
@@
 	)
 	(segment
-		(start 122.25051 121.14274)
-		(end 120.80051 119.69274)
-		(width 0.2)
-		(layer "F.Cu")
-		(net "GND")
-	)
-	(segment
 		(start 125.40051 104.39274)
 		(end 125.40051 104.14274)
@@
 	)
 	(segment
-		(start 122.25051 121.29274)
-		(end 122.25051 121.14274)
-		(width 0.2)
-		(layer "F.Cu")
-		(net "GND")
-	)
-	(segment
 		(start 124.28801 113.89274)
 		(end 124.43801 113.74274)
@@
 	)
 	(segment
+		(start 120.80051 119.94274)
+		(end 120.80051 115.49274)
+		(width 0.2)
+		(layer "F.Cu")
+		(net "GND")
+	)
+	(segment
 		(start 123.35051 84.13024)
 		(end 123.31301 84.09274)
@@
 	)
 	(via
-		(at 132.53801 86.79274)
+		(at 132.45051 86.34274)
 		(size 0.6)
 		(drill 0.3)
@@
 	)
 	(segment
-		(start 116.10051 83.377054)
-		(end 116.10051 81.34274)
-		(width 0.25)
-		(layer "F.Cu")
-		(net "+5V")
-	)
-	(segment
-		(start 116.10051 81.34274)
-		(end 114.95051 80.19274)
+		(start 106.90051 86.24274)
+		(end 105.55051 87.59274)
 		(width 0.25)
 		(layer "F.Cu")
@@
 	)
 	(segment
-		(start 106.90051 86.24274)
-		(end 105.55051 87.59274)
-		(width 0.25)
-		(layer "F.Cu")
-		(net "+5V")
-	)
-	(segment
 		(start 130.10051 103.49274)
 		(end 130.10051 103.44274)
@@
 	)
 	(segment
-		(start 108.85051 80.19274)
-		(end 106.90051 82.14274)
-		(width 0.25)
-		(layer "F.Cu")
-		(net "+5V")
-	)
-	(segment
 		(start 124.80051 101.89274)
 		(end 122.95051 101.89274)
@@
 	)
 	(segment
+		(start 116.91301 85.65524)
+		(end 115.75051 84.49274)
+		(width 0.2)
+		(layer "F.Cu")
+		(net "+5V")
+	)
+	(segment
+		(start 117.20051 85.65524)
+		(end 116.91301 85.65524)
+		(width 0.2)
+		(layer "F.Cu")
+		(net "+5V")
+	)
+	(segment
 		(start 119.48801 98.730239)
 		(end 117.21301 98.730239)
@@
 	)
 	(segment
-		(start 117.46301 84.739554)
-		(end 116.10051 83.377054)
+		(start 115.75051 83.09274)
+		(end 115.75051 80.99274)
 		(width 0.25)
 		(layer "F.Cu")
@@
 	)
 	(segment
-		(start 100.75727 86.5495)
-		(end 100.75727 86.54274)
-		(width 0.2)
+		(start 115.75051 80.99274)
+		(end 114.95051 80.19274)
+		(width 0.25)
 		(layer "F.Cu")
 		(net "+5V")
@@
 	)
 	(segment
-		(start 117.46301 85.65524)
-		(end 117.46301 84.739554)
+		(start 106.90051 82.14274)
+		(end 106.90051 86.24274)
 		(width 0.25)
 		(layer "F.Cu")
@@
 	)
 	(segment
-		(start 106.90051 82.14274)
-		(end 106.90051 86.24274)
-		(width 0.25)
-		(layer "F.Cu")
-		(net "+5V")
-	)
-	(segment
 		(start 101.38426 74.96899)
 		(end 101.38426 81.268988)
@@
 	)
 	(segment
+		(start 115.75051 84.49274)
+		(end 115.75051 83.09274)
+		(width 0.2)
+		(layer "F.Cu")
+		(net "+5V")
+	)
+	(segment
 		(start 119.788009 98.730239)
 		(end 119.48801 98.730239)
@@
 	)
 	(segment
+		(start 114.95051 80.19274)
+		(end 108.85051 80.19274)
+		(width 0.25)
+		(layer "F.Cu")
+		(net "+5V")
+	)
+	(segment
 		(start 101.69426 89.536491)
 		(end 101.65051 89.580241)
@@
 	)
 	(segment
+		(start 108.85051 80.19274)
+		(end 106.90051 82.14274)
+		(width 0.25)
+		(layer "F.Cu")
+		(net "+5V")
+	)
+	(segment
 		(start 100.80676 82.18649)
 		(end 100.80676 83.93649)
@@
 	)
 	(segment
-		(start 114.95051 80.19274)
-		(end 108.85051 80.19274)
-		(width 0.25)
-		(layer "F.Cu")
-		(net "+5V")
-	)
-	(segment
 		(start 128.60051 104.89274)
 		(end 128.70051 104.89274)
@@
 	)
 	(segment
-		(start 119.15051 121.29274)
+		(start 119.15051 121.54274)
 		(end 119.15051 119.29274)
 		(width 0.2)
@@
 	)
 	(segment
+		(start 119.20051 121.59274)
+		(end 119.15051 121.54274)
+		(width 0.2)
+		(layer "F.Cu")
+		(net "NXP_TPSOUT02")
+	)
+	(segment
 		(start 126.585125 138.505114)
 		(end 128.457865 138.505114)
@@
 	)
 	(segment
-		(start 135.40051 72.59274)
-		(end 136.55051 72.59274)
-		(width 0.7)
-		(layer "F.Cu")
-		(net "unconnected-(K1-Pad2)")
-	)
-	(segment
